File: hardware/nonstandard/nonstandard.kicad_sch (KiCad schematic)
At the start: 0 parts

Commit message: Update KiCad project configuration defaults
Parts:
- added C1, C22, C48: 47n, symbol Device:C
- added C10, C26, C30, C33, C36, C6: 20n, symbol Device:C
- added C11, C19, C20, C3, C32, C39: 100u, symbol Device:C_Polarized
- added C12: 250p, symbol Device:C
- added C13, C14, C35: 50n, symbol Device:C
- added C15, C28: 10n, symbol Device:C
- added C16, C2, C25, C38: 180p, symbol Device:C
- added C17, C18, C34, C40, C5, C7: 2u, symbol Device:C_Polarized
- added C21, C31, C4, C9: 39p, symbol Device:C
- added C23, C27: 25u, symbol Device:C_Polarized
- added C24: 220n, symbol Device:C
- added C29, C37, C41, C56, C8: 100n, symbol Device:C
- added C42: 200p, symbol Device:C
- added C43, C44, C45, C51, C62: 2u, symbol Device:C
- added C46: 5p, symbol Device:C
- added C47, C49: 2.2n, symbol Device:C
- added C50: 82p, symbol Device:C
- added C52: 10u, symbol Device:C_Polarized
- added C53, C59, C60: 2.2u, symbol Device:C
- added C54: 33p, symbol Device:C
- added C55: 22n, symbol Device:C
- added C57: 5n, symbol Device:C
- added C58: 8.2n, symbol Device:C
- added C61: 27n, symbol Device:C
- added D1, D2, D3, D4, D5, D6: D, symbol Device:D
- added Q1, Q10, Q11, Q12, Q14, Q15, Q2, Q4, Q7, Q9: NPN, symbol Simulation_SPICE:NPN
- added Q13, Q3, Q5, Q8: PNP, symbol Simulation_SPICE:PNP
- added Q6: NJFET, symbol Simulation_SPICE:NJFET
- added R1, R16, R26, R30, R34, R38, R47, R52, R54, R57, R8, R81: 4.7K, symbol Device:R
- added R10, R56, R73, R74: 22K, symbol Device:R
- added R11, R15, R23, R27, R32, R35, R42, R48, R7: 2.7K, symbol Device:R
- added R12, R17, R22, R28, R31, R4, R44, R46, R6, R61, R62, R67: 47K, symbol Device:R
- added R13, R2, R33, R45, R66, R84, R86: 1M, symbol Device:R
- added R14, R58, R64, R68, R70, R77: 100K, symbol Device:R
- added R18, R20, R25, R49, R53, R71, R79: 10K, symbol Device:R
- added R19, R72, R75: 68K, symbol Device:R
- added R21, R24, R39, R50, R60: 100R, symbol Device:R
- added R29, R3, R76: 470K, symbol Device:R
- added R36, R40, R80, R91: 15K, symbol Device:R
- added R37, R59, R9: 330R, symbol Device:R
- added R41: 680R, symbol Device:R
- added R43, R92: 220K, symbol Device:R
- added R5, R51, R55: 1K, symbol Device:R
- added R63: 2.2M, symbol Device:R
- added R65, R78: 120K, symbol Device:R
- added R69, R83: 330K, symbol Device:R
- added R82, R88, R89: 12K, symbol Device:R
- added R85: 1.5K, symbol Device:R
- added R87: 33K, symbol Device:R
- added R90: 3.3K, symbol Device:R
- added R93: 150R, symbol Device:R
- added RV1, RV5, RV6, RV7, RV8: 10K, symbol Device:R_Potentiometer
- added RV10, RV2, RV9: 50K, symbol Device:R_Potentiometer
- added RV11, RV12: 1MB, symbol Device:R_Potentiometer
- added RV13, RV14, RV15, RV16: 100KB, symbol Device:R_Potentiometer
- added RV3, RV4: 250K, symbol Device:R_Potentiometer
- added U1: 74HC04, symbol 74xx:74HC04
- added U2, U3, U4, U5: Opamp_Dual, symbol Device:Opamp_Dual
Connections:
- new net: R9.1, RV1.1
- new net: C5.2, R9.2
- new net: C4.2, Q2.2 (B), Q3.1 (C), R6.2
- new net: C28.1, R27.1, R32.1, RV5.3
- new net: C23.2, D1.1 (K), D2.2 (A), R32.2
- new net: C20.1, Q8.3 (E), Q9.1 (C), R28.2, R29.2, R39.2
- new net: C1.2, Q1.2 (B), R2.2, R3.1
- new net: C23.1, Q9.3 (E), R35.2, R36.1
- new net: C27.1, Q10.3 (E), R34.2, R36.2
- new net: C10.2, R15.1
- new net: Q4.3 (E), R15.2, R16.2, R17.2
- new net: C62.2, R93.2
- new net: C26.2, R34.1
- new net: R57.1, R58.1, R59.2
- new net: R53.1, RV9.2
- new net: C36.1, C37.1, C41.2, R53.2
- new net: R87.1, R89.2, U4.6 (-)
- new net: R87.2, R88.1, U4.7
- new net: C16.1, Q6.1 (D), Q7.2 (B), R22.1
- new net: Q11.3 (E), R41.2, R42.1
- new net: D1.2 (A), D2.1 (K), R42.2
- new net: C18.1, Q7.3 (E), R26.2
- new net: C59.1, R86.1, RV14.3, U4.5 (+)
- new net: Q6.2 (G), RV4.2
- new net: Q6.3 (S), R23.2
- new net: C38.2, C39.1, Q15.1 (C), R50.1, R56.2, R60.2
- new net: D5.2 (A), D6.1 (K), R92.2, R93.1, U5.1
- new net: Q11.2 (B), R43.1
- new net: C11.1, Q2.1 (C), Q5.3 (E), R12.2, R13.2, R24.2, R5.1
- new net: C7.1, Q2.3 (E), R10.1, R7.2
- new net: C14.1, C15.2, RV2.1, RV2.2
- new net: C13.1, C14.2, R19.1
- new net: C51.1, R76.1, U1.9
- new net: C52.1, R76.2, U1.8
- new net: C50.2, R72.1, R73.2, U1.5
- new net: C49.2, R71.2, R72.2, U1.6
- new net: C6.2, R8.1
- new net: C53.1, C55.2, R79.1, R80.1
- new net: C53.2, C54.1, R78.2, U3.1
- new net: C1.1, C2.2, R1.2
- new net: R37.1, RV5.1
- new net: C27.2, R37.2, R40.1, RV8.3
- new net: C30.2, D3.1 (K), D4.2 (A), R40.2
- new net: C38.1, Q14.1 (C), Q15.2 (B), R56.1
- new net: C48.2, R67.2, R69.1, R70.1, U1.1
- new net: R70.2, RV12.1
- new net: C37.2, Q14.2 (B), R58.2
- new net: R64.2, RV11.1
- new net: C45.2, RV11.2
- new net: R65.1, RV11.3
- new net: C21.2, Q8.1 (C), Q9.2 (B), R31.2
- new net: C21.1, Q10.1 (C), Q8.2 (B), R28.1
- new net: R55.2, RV10.1
- new net: C36.2, RV10.2
- new net: R51.2, RV10.3
- new net: C61.1, R90.2, R91.1
- new net: R91.2, RV15.2
- new net: R89.1, RV14.1
- new net: C60.2, RV14.2
- new net: R69.2, R74.1, U1.2
- new net: C35.1, R52.1, RV9.1
- new net: C34.2, R51.1, R52.2
- new net: C22.1, C25.2, R30.2
- new net: C22.2, Q10.2 (B), R29.1, R33.2
- new net: R27.2, RV6.1
- new net: C3.1, Q3.3 (E), R3.2, R4.2, R5.2
- new net: C57.1, C58.1, C59.2, R83.2, R85.2
- new net: C50.1, R71.1
- new net: C52.2, R77.1
- new net: C47.2, R67.1
- new net: C55.1, R80.2, R81.2, U3.5 (+)
- new net: C43.1, C44.2, R63.1, R64.1, U2.2 (-)
- new net: C34.1, Q13.1 (C), R46.1, R49.2
- new net: C33.2, R48.1
- new net: Q12.3 (E), R46.2, R47.2, R48.2
- new net: R88.2, R92.1, RV13.1, RV15.1, RV16.1, RV16.2, U5.2 (-)
- new net: C7.2, R11.2
- new net: C49.1, RV12.2
- new net: C8.2, R11.1, RV1.3
- new net: C56.1, R79.2, R82.2, RV13.2
- new net: C4.1, Q1.1 (C), Q3.2 (B), R4.1
- new net: C24.1, RV7.3
- new net: C35.2, R54.1, RV9.3
- new net: C5.1, Q1.3 (E), R10.2, R8.2
- new net: C8.1, C9.1, Q4.2 (B), R13.1, R14.2
- new net: C44.1, C45.1, R63.2, U2.1
- new net: C12.1, Q5.1 (C), R17.1, R18.2, R19.2
- new net: C9.2, Q4.1 (C), Q5.2 (B), R12.1
- new net: C29.2, C31.1, Q12.2 (B), R45.1
- new net: C32.1, Q13.3 (E), R39.1, R44.2, R45.2, R50.2
- new net: C28.2, C29.1, R38.1
- new net: C31.2, Q12.1 (C), Q13.2 (B), R44.1
- new net: C40.1, Q15.3 (E), R57.2
- new net: C46.1, R65.2, R66.1, U2.6 (-)
- new net: C46.2, C47.1, R66.2, R68.1, U2.7
- new net: C24.2, R38.2, RV6.2, RV6.3
- new net: C48.1, R68.2
- new net: C58.2, R84.2, U4.3 (+)
- new net: R20.2, RV3.2, RV3.3
- new net: C43.2, R62.2
- new net: R73.1, R75.2, U1.4
- new net: R85.1, U4.1, U4.2 (-)
- new net: R74.2, R75.1, U1.3
- new net: C13.2, R21.1, RV3.1
- new net: R21.2, RV4.3
- new net: Q11.1 (C), RV8.2
- new net: C42.2, R61.2, R62.1
- new net: C12.2, RV4.1
- new net: C51.2, RV12.3
- new net: C17.1, R23.1, R25.2
- new net +15V: D5.1 (K)
- new net +24V: C16.2, C19.1, Q7.1 (C), R22.2, R24.1, R60.1
- new net -15V: D6.2 (A)
- new net DIST_ENABLE: R43.2
- new net FX_LOOP: C62.1, RV16.3
- new net GND: C10.1, C11.2, C15.1, C17.2, C19.2, C2.1, C20.2, C25.1, C26.1, C3.2, C30.1, C32.2, C33.1, C39.2, C41.1, C42.1, C56.2, C57.2, C6.1, C60.1, D3.2 (A), D4.1 (K), Q14.3 (E), R14.1, R16.1, R18.1, R2.1, R20.1, R25.1, R26.1, R31.1, R33.1, R35.1, R41.1, R47.1, R49.1, R59.1, R6.1, R7.1, R81.1, R82.1, R84.1, R86.2, R90.1, RV1.2, RV13.3, RV15.3, RV2.3, RV5.2, RV7.1, RV7.2, RV8.1, U2.3 (+), U2.5 (+), U3.3 (+), U5.3 (+)
- new net IN: R1.1, R30.1, R61.1
- new net SUMMING_AMP: C18.2, C40.2, R54.2, R55.1
- new net SW_FETS_SKIPPED: C54.2, R77.2, R78.1, U3.2 (-)
- new net TO_RVB: C61.2, R83.1, U3.6 (-), U3.7
Other:
- note added: "0.6V"
- note added: "0.7V"
- note added: "0V"
- note added: "1.4V"
- note added: "1.8V"
- note added: "12.6V"
- note added: "12V"
- note added: "13.4V"
- note added: "13.6V"
- note added: "13V"
- note added: "14V"
- note added: "15V"
- note added: "20.4V"
- note added: "21.4V"
- note added: "21V"
- note added: "22V"
- note added: "2V"
- note added: "Distortion"
- note added: "Gain stage"
- note added: "Preamp"
- note added: "Tone amp"

Commit message: Add digital hardware schematic
Parts:
- removed C1, C22, C48: 47n, symbol Device:C
- removed C10, C26, C30, C33, C36, C6: 20n, symbol Device:C
- removed C11, C19, C20, C3, C32, C39: 100u, symbol Device:C_Polarized
- removed C12: 250p, symbol Device:C
- removed C13, C14, C35: 50n, symbol Device:C
- removed C15, C28: 10n, symbol Device:C
- removed C16, C2, C25, C38: 180p, symbol Device:C
- removed C17, C18, C34, C40, C5, C7: 2u, symbol Device:C_Polarized
- removed C21, C31, C4, C9: 39p, symbol Device:C
- removed C23, C27: 25u, symbol Device:C_Polarized
- removed C24: 220n, symbol Device:C
- removed C29, C37, C41, C56, C8: 100n, symbol Device:C
- removed C42: 200p, symbol Device:C
- removed C43, C44, C45, C51, C62: 2u, symbol Device:C
- removed C46: 5p, symbol Device:C
- removed C47, C49: 2.2n, symbol Device:C
- removed C50: 82p, symbol Device:C
- removed C52: 10u, symbol Device:C_Polarized
- removed C53, C59, C60: 2.2u, symbol Device:C
- removed C54: 33p, symbol Device:C
- removed C55: 22n, symbol Device:C
- removed C57: 5n, symbol Device:C
- removed C58: 8.2n, symbol Device:C
- removed C61: 27n, symbol Device:C
- removed D1, D2, D3, D4, D5, D6: D, symbol Device:D
- removed Q1, Q10, Q11, Q12, Q14, Q15, Q2, Q4, Q7, Q9: NPN, symbol Simulation_SPICE:NPN
- removed Q13, Q3, Q5, Q8: PNP, symbol Simulation_SPICE:PNP
- removed Q6: NJFET, symbol Simulation_SPICE:NJFET
- removed R1, R16, R26, R30, R34, R38, R47, R52, R54, R57, R8, R81: 4.7K, symbol Device:R
- removed R10, R56, R73, R74: 22K, symbol Device:R
- removed R11, R15, R23, R27, R32, R35, R42, R48, R7: 2.7K, symbol Device:R
- removed R12, R17, R22, R28, R31, R4, R44, R46, R6, R61, R62, R67: 47K, symbol Device:R
- removed R13, R2, R33, R45, R66, R84, R86: 1M, symbol Device:R
- removed R14, R58, R64, R68, R70, R77: 100K, symbol Device:R
- removed R18, R20, R25, R49, R53, R71, R79: 10K, symbol Device:R
- removed R19, R72, R75: 68K, symbol Device:R
- removed R21, R24, R39, R50, R60: 100R, symbol Device:R
- removed R29, R3, R76: 470K, symbol Device:R
- removed R36, R40, R80, R91: 15K, symbol Device:R
- removed R37, R59, R9: 330R, symbol Device:R
- removed R41: 680R, symbol Device:R
- removed R43, R92: 220K, symbol Device:R
- removed R5, R51, R55: 1K, symbol Device:R
- removed R63: 2.2M, symbol Device:R
- removed R65, R78: 120K, symbol Device:R
- removed R69, R83: 330K, symbol Device:R
- removed R82, R88, R89: 12K, symbol Device:R
- removed R85: 1.5K, symbol Device:R
- removed R87: 33K, symbol Device:R
- removed R90: 3.3K, symbol Device:R
- removed R93: 150R, symbol Device:R
- removed RV1, RV5, RV6, RV7, RV8: 10K, symbol Device:R_Potentiometer
- removed RV10, RV2, RV9: 50K, symbol Device:R_Potentiometer
- removed RV11, RV12: 1MB, symbol Device:R_Potentiometer
- removed RV13, RV14, RV15, RV16: 100KB, symbol Device:R_Potentiometer
- removed RV3, RV4: 250K, symbol Device:R_Potentiometer
- removed U1: 74HC04, symbol 74xx:74HC04
- removed U2, U3, U4, U5: Opamp_Dual, symbol Device:Opamp_Dual
Other:
- added sheet digi (digi.kicad_sch)
- added sheet peavey_dist (peavey_dist.kicad_sch)
- added sheet peavey_normal (peavey_normal.kicad_sch)
- added sheet power (power.kicad_sch)
- added sheet power_amp (power_amp.kicad_sch)
- added sheet preamp (preamp.kicad_sch)
- added sheet sunn (sunn.kicad_sch)
- note removed: "0.6V"
- note removed: "0.7V"
- note removed: "0V"
- note removed: "1.4V"
- note removed: "1.8V"
- note removed: "12.6V"
- note removed: "12V"
- note removed: "13.4V"
- note removed: "13.6V"
- note removed: "13V"
- note removed: "14V"
- note removed: "15V"
- note removed: "20.4V"
- note removed: "21.4V"
- note removed: "21V"
- note removed: "22V"
- note removed: "2V"
- note removed: "Distortion"
- note removed: "Gain stage"
- note removed: "Preamp"
- note removed: "Tone amp"
