File: hardware/nonstandard/digi.kicad_sch (KiCad schematic)
At the start: 13 parts, among them J1 LCD, SW1 VOL, SW2 MOON, SW3 SUNN, SW4 BASS, SW5 MID, SW6 TREBLE, SW7 MASTER, U11 MCP23S17_ML

Commit message: Update digital schematic layout and add display documentation
Parts:
- added C2: 100n, symbol Device:C
- added R1, R3: 10K, symbol Device:R
- added U2: MCP23S17_ML, Package_DFN_QFN:QFN-28-1EP_6x6mm_P0.65mm_EP4.25x4.25mm, symbol Interface_Expansion:MCP23S17_ML
- J1: footprint (none) -> nonstandard:4004
- SW1, SW2, SW3, SW4, SW5, SW6, SW7: footprint (none) -> Rotary_Encoder:RotaryEncoder_Alps_EC11E-Switch_Vertical_H20mm
- renumbered C103 to C1, R129 to R2, RV17 to RV1, U11 to U1
Connections:
- net +3.3V: now also C2.1, R1.2, R3.2, U2.11 (A0), U2.5 (VDD)
- net GND: now also C2.2, U2.12 (A1), U2.13 (A2), U2.29 (EP), U2.6 (VSS)
- net MCP_CS: now also U2.7 (~{CS})
- net MCP_INT: now also R1.1, U2.16 (INTA)
- net MCP_SCK: now also U2.8 (SCK)
- net MCP_SI: now also U2.9 (SI)
- net MCP_SO: now also U2.10 (SO)
- net SW1: now also U2.17 (GPA0); no longer A1.21 (GPIO16)
- net SW2: now also U2.18 (GPA1); no longer A1.22 (GPIO17)
- net SW3: now also U2.19 (GPA2); no longer A1.24 (GPIO18)
- net SW4: now also U2.20 (GPA3); no longer A1.25 (GPIO19)
- net SW5: now also U2.21 (GPA4); no longer A1.26 (GPIO20)
- net SW6: now also U2.22 (GPA5); no longer A1.27 (GPIO21)
- net SW7: now also U2.23 (GPA6); no longer A1.29 (GPIO22)
- new net: R3.1, U2.14 (~{RESET})
Other:
- moved on the sheet: A1, C1, R2, SW1, SW2, SW3, SW4, SW5, SW6, SW7, U1
