File: hardware/nonstandard/peavey_dist.kicad_sch (KiCad schematic)
At the start: 74 parts, among them Q10 NPN, Q11 NPN, Q12 NPN, Q13 PNP, Q14 NPN, Q15 NPN, Q8 PNP, Q9 NPN

Commit message: Update digital schematic layout and add display documentation
Parts:
- renumbered C20 to C22, C32 to C23, C39 to C24, C38 to C25, C28 to C26, C31 to C27, C36 to C28, C21 to C29, C22 to C30, C40 to C31, C23 to C32, C29 to C33, C25 to C34, C37 to C35, C34 to C36, C24 to C37, C26 to C38, C41 to C39, C33 to C40, C27 to C41, C35 to C42, C30 to C43, D2 to D1, D1 to D2, D4 to D3, D3 to D4, Q15 to Q10, Q9 to Q11, Q10 to Q12, Q12 to Q13, Q11 to Q15, Q13 to Q9, R39 to R30, R50 to R31, R60 to R32, R28 to R33, R45 to R34, R44 to R35, R56 to R36, R29 to R37, R51 to R38, R55 to R39, R30 to R40, R31 to R41, R32 to R42, R27 to R43, R38 to R44, R33 to R45, R34 to R46, R35 to R47, R46 to R48, R48 to R49, R57 to R50, R36 to R51, R58 to R55, R47 to R56, R49 to R57, R59 to R58, R37 to R59, R40 to R60, R42 to R61, R43 to R62, R41 to R63, RV5 to RV10, RV8 to RV11, RV10 to RV6, RV6 to RV7, RV7 to RV8
