File: hardware/nonstandard/peavey_normal.kicad_sch (KiCad schematic)
At the start: 56 parts, among them Q1 NPN, Q2 NPN, Q3 PNP, Q4 NPN, Q5 PNP, Q6 NJFET, Q7 NPN

Commit message: Update digital schematic layout and add display documentation
Parts:
- renumbered C1 to C10, C7 to C11, C8 to C12, C18 to C13, C2 to C14, C13 to C15, C6 to C16, C14 to C17, C5 to C18, C10 to C19, C15 to C20, C17 to C21, C11 to C4, C19 to C5, C16 to C6, C12 to C7, C9 to C8, C4 to C9, Q3 to Q1, Q7 to Q2, Q5 to Q3, Q6 to Q4, Q2 to Q5, Q1 to Q6, Q4 to Q7, R3 to R10, R1 to R11, R6 to R12, R11 to R13, R19 to R14, R21 to R15, R2 to R16, R8 to R17, R7 to R18, R17 to R19, R23 to R20, R26 to R21, R10 to R22, R14 to R23, R16 to R24, R15 to R25, R18 to R26, R20 to R27, R25 to R28, R9 to R29, R5 to R4, R24 to R5, R4 to R6, R22 to R7, R13 to R8, R12 to R9, RV4 to RV2, RV2 to RV4, RV1 to RV5
