File: hardware/nonstandard/power.kicad_sch (KiCad schematic)
At the start: 30 parts, among them J2 HV +, J3 LV +, J4 HV -, J5 LV -, J6 HV CT, U7 LMR36510ADDA, U8 LM7808_TO220, U9 LM7824_TO220

Commit message: Update digital schematic layout and add display documentation
Parts:
- renumbered C88 to C65, C91 to C66, C89 to C67, C90 to C68, C92 to C69, C93 to C70, C94 to C71, C95 to C72, C98 to C73, C64 to C74, C96 to C75, C97 to C76, C102 to C77, C99 to C78, C101 to C79, C70 to C80, C100 to C81, D12 to D7, D11 to D8, J3 to J2, J5 to J3, J2 to J4, J4 to J5, R100 to R97, R101 to R98, U7 to U10, U9 to U8, U8 to U9
