File: hardware/nonstandard/preamp.kicad_sch (KiCad schematic)
At the start: 73 parts, among them Q16 PNP, Q17 NPN, Q18 NPN, Q19 NPN, Q20 NPN, Q21 NJFET, U6 74C04

Commit message: Update digital schematic layout and add display documentation
Parts:
- removed C63, C80: 100u, symbol Device:C_Polarized
- removed C65: 39p, symbol Device:C
- removed C66, C79: 47n, symbol Device:C
- removed C67, C72: 25u, symbol Device:C_Polarized
- removed C68: 100n, symbol Device:C
- removed C69, C81: 180p, symbol Device:C
- removed C71, C73: 20n, symbol Device:C
- removed C74: 2u, symbol Device:C
- removed C75: 10u, symbol Device:C_Polarized
- removed C76, C77: 2.2n, symbol Device:C
- removed C78: 82p, symbol Device:C
- removed C82: 250p, symbol Device:C
- removed C83, C87: 2u, symbol Device:C_Polarized
- removed C84: 50n, symbol Device:C
- removed D7, D8: D, symbol Device:D
- removed R94: 100R, symbol Device:R
- removed R95, R98: 47K, symbol Device:R
- removed R96: 470K, symbol Device:R
- removed R97: 4.7K, symbol Device:R
- removed RV24: 50K, symbol Device:R_Potentiometer
- removed U6: 74C04, symbol 74xx:74HC04
- added C100: 250p, symbol Device:C
- added C101, C105: 2u, symbol Device:C_Polarized
- added C102, C103: 50n, symbol Device:C
- added C104: 10n, symbol Device:C
- added C82, C98: 100u, symbol Device:C_Polarized
- added C83: 2u, symbol Device:C
- added C84: 10u, symbol Device:C_Polarized
- added C87, C90: 2.2n, symbol Device:C
- added C88, C95: 25u, symbol Device:C_Polarized
- added C89, C96: 100n, symbol Device:C
- added C91: 82p, symbol Device:C
- added C92, C99: 180p, symbol Device:C
- added C93: 47n, symbol Device:C
- added C94, C97: 20n, symbol Device:C
- added D11, D12: D, symbol Device:D
- added R100: 47K, symbol Device:R
- added R101: 470K, symbol Device:R
- added R129: 2.7K, symbol Device:R
- added R130: 4.7K, symbol Device:R
- added R131, R132: 10K, symbol Device:R
- added RV18: 1MB, symbol Device:R_Potentiometer
- added U11: 4069UB, Package_DIP:CERDIP-14_W7.62mm_SideBrazed_Socket, symbol 4xxx:4069
- C85: value 50n -> 39p
- C86: value 10n -> 47n
- R102: value 1M -> 470K
- R103: value 4.7K -> 100K
- R104: value 2.7K -> 100K
- R105: value 15K -> 4.7K
- R106: value 330R -> 47K
- R107: value 15K -> 2.7K
- R108: value 2.7K -> 47K
- R109: value 220K -> 330K
- R110: value 680R -> 68K
- R111: value 470K -> 10K
- R112: value 100K -> 1M
- R113: value 47K -> 4.7K
- R114: value 330K -> 2.7K
- R115: value 68K -> 100K
- R116: value 10K -> 22K
- R117: value 100K -> 22K
- R118: value 22K -> 68K
- R119: value 22K -> 15K
- R120: value 68K -> 330R
- R121: value 100R -> 15K
- R122: value 47K -> 2.7K
- R123: value 68K -> 220K
- R124: value 100R -> 680R
- R125, R99: value 2.7K -> 100R
- R126: value 4.7K -> 47K
- R127: value 10K -> 68K
- R128: value 10K -> 100R
- RV21: value 1MB -> 250K
- RV23: value 250K -> 50K
Connections:
- net +24V: now also R125.1, R126.2, C98.1, C99.2; no longer R121.1, R122.2
- net DIST_ENABLE: now also R123.2; no longer R109.2
- net GND: now also R106.1, R112.1, R114.1, R124.1, RV23.3, C104.1, C105.2, C82.2, C92.1, C94.1, C96.2, C97.1, C98.2, D11.1 (K), D12.2 (A), R130.1, R131.1, R132.1, U11.11, U11.13, U11.14 (VDD); no longer C86.1, D10.2 (A), D9.1 (K), R102.1, R104.1, R110.1, R126.1, R127.1, R128.1
- net at R128.2: now also RV21.3; no longer R125.1
- net at R117.1: now also R110.2, U11.4
- net at R113.1: now also C94.2
- net at Q20.2 (B), Q21.1 (D): now also R126.1, C99.1; no longer R122.1
- net at Q20.3 (E): now also C101.1, R130.2; no longer R126.2
- net at R114.2: now also Q17.3 (E), R119.1, C88.1; no longer R118.1
- net at R109.1: now also R103.1, R108.2, C93.2, U11.1; no longer Q19.2 (B)
- net at RV21.2: now also Q21.2 (G)
- net at R120.2: now also R121.1, RV20.3, C95.2; no longer R116.2
- net at Q16.3 (E), Q17.1 (C): now also R102.2, R99.2, C82.1, R100.2
- net at C85.1: now also Q16.2 (B), Q18.1 (C), R100.1; no longer C86.2
- net at R119.2: now also Q18.3 (E), R113.2, C95.1; no longer R120.1
- net at Q16.1 (C), Q17.2 (B): now also C85.2, R106.2
- net at R123.1: now also Q19.2 (B); no longer C85.2
- net at RV23.1: now also RV23.2, C103.1, C104.2; no longer R124.1
- net at R111.2: now also R118.2, C87.2, U11.6
- net at R111.1: now also C91.1
- net at RV22.2: now also RV22.3, R131.2; no longer Q21.2 (G)
- net at Q21.3 (S): now also R129.2; no longer R125.2
- net at R124.2: now also Q19.3 (E), R122.1; no longer RV22.3
- net at R117.2: now also R118.1, C91.2, U11.5
- net at R115.1: now also C90.1; no longer R118.2
- net at R115.2: now also C93.1; no longer R119.1
- net at Q18.2 (B): now also C86.2, R102.1, R112.2; no longer R102.2
- net at RV22.1: now also R128.1, C102.2
- net at RV19.3: now also R107.1, C89.1; no longer R99.1
- net at D10.1 (K), D9.2 (A), R107.2: now also C88.2
- net at RV19.1: now also R120.1; no longer R106.1
- net at R121.2: now also C97.2, D11.2 (A), D12.1 (K)
- net at R116.1: now also R109.2, U11.2
- net at RV21.1: now also C100.2; no longer R112.2
- new net: C90.2, R108.1
- new net: R103.2, RV18.1
- new net: C87.1, RV18.2
- new net: C83.2, RV18.3
- new net: C105.1, R129.1, R132.2
- new net: C102.1, C103.2, R127.1
- new net: C83.1, R101.1, U11.9
- new net: C84.1, R101.2, U11.8
- new net: C100.1, R127.2
- new net: C84.2, R104.1
- new net: D10.2 (A), D9.1 (K), R122.2
- new net: C86.1, C92.2, R105.2
- new net: R110.1, R116.2, U11.3
- new net +8V: C96.1, U11.7 (VSS)
- new net IN: R105.1
- now unconnected: R104.2
- no-connect marks 0 -> 2
Other:
- note added: "FX Loop"
- note added: "Interstage Control"
- note added: "Line Out"
- note added: "Peavey Distortion"
- note added: "Peavey Preamp"
- note added: "Sunn Distortion"
- note removed: "Distortion"
- note removed: "Preamp"
