File: hardware/nonstandard/sunn.kicad_sch (KiCad schematic)
At the start: 67 parts, among them U10 4069UB, U2 Opamp_Dual, U3 Opamp_Dual, U4 Opamp_Dual, U5 Opamp_Dual

Commit message: Update digital schematic layout and add display documentation
Parts:
- U3: renamed from U10; footprint (none) -> Package_DIP:CERDIP-14_W7.62mm_SideBrazed_Socket
- U4: renamed from U2; footprint (none) -> Package_DIP:CERDIP-8_W7.62mm_SideBrazed_Socket
- U5: renamed from U3; footprint (none) -> Package_DIP:CERDIP-8_W7.62mm_SideBrazed_Socket
- U6: renamed from U4; footprint (none) -> Package_DIP:CERDIP-8_W7.62mm_SideBrazed_Socket
- U7: renamed from U5; footprint (none) -> Package_DIP:CERDIP-8_W7.62mm_SideBrazed_Socket
- renumbered C51 to C44, C52 to C45, C45 to C47, C49 to C48, C47 to C49, C44 to C51, C48 to C52, C43 to C53, C42 to C54, C54 to C55, C55 to C57, C53 to C58, C57 to C60, C58 to C61, C60 to C63, C61 to C64, R76 to R64, R70 to R65, R77 to R66, R64 to R67, R65 to R68, R63 to R69, R66 to R70, R67 to R71, R69 to R72, R75 to R73, R71 to R74, R68 to R75, R74 to R76, R73 to R77, R72 to R78, R61 to R79, R62 to R80, R79 to R81, R78 to R83, R86 to R84, R92 to R85, R80 to R86, R83 to R87, R81 to R89, R93 to R90, R85 to R91, R87 to R92, R89 to R93, R84 to R94, R91 to R95, R90 to R96, RV11 to RV13, RV13 to RV14, RV16 to RV15, RV14 to RV16, RV15 to RV17
